Commit message: rviz robot display

File: src/ur5_pybullet_ros/script/urdf/ur5_robotiq_85_rviz.urdf (robot description, URDF)
Before this commit: robot ur5_robotiq_85, 20 links, 19 joints
Links:
- link base_link: geometry collision mesh filename=package://ur5_pybullet_ros/script/meshes/ur5/collision/base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; visual mesh filename=package://ur5_pybullet_ros/script/meshes/ur5/visual/base.stl
