Commit message: chassis

File: src/ur5_pybullet_ros/script/urdf/ur5_robotiq_85_mobile.urdf (robot description, URDF)
Before this commit: robot ur5_robotiq_85, 20 links, 19 joints
Links:
- added link chassis_link, mass 20.0; collision box size=0.5 0.5 0.1; visual box size=0.5 0.5 0.1
- added link chassis_link_theta, mass 0
- added link chassis_link_x, mass 0
- added link chassis_link_y, mass 0
- added link lidar_link, mass 40.0; visual cylinder length=0.02 radius=0.03
Joints:
- removed joint world_arm_joint
- added joint chassis_joint: type fixed, parent chassis_link, child base_link, origin xyz=0.0 0.0 0.1 rpy=0.0 0.0 0.0
- added joint lidar_joint: type fixed, parent chassis_link, child lidar_link, origin xyz=0.2 0.0 0.1 rpy=0.0 0.0 0.0
- added joint world_chassis_joint_fixed: type fixed, parent chassis_link_theta, child chassis_link, origin xyz=0 0 0 rpy=0.0 0.0 0
- added joint world_chassis_joint_theta: type continuous, parent chassis_link_y, child chassis_link_theta, origin xyz=0 0 0 rpy=0.0 0.0 0, axis 0 0 1
- added joint world_chassis_joint_x: type prismatic, parent world, child chassis_link_x, origin xyz=0 0 0 rpy=0.0 0.0 0, axis 1 0 0, limit lower=-100 upper=100 effort=5000 velocity=3
- added joint world_chassis_joint_y: type prismatic, parent chassis_link_x, child chassis_link_y, origin xyz=0 0 0 rpy=0.0 0.0 0, axis 0 1 0, limit lower=-100 upper=100 effort=5000 velocity=3

Commit message: cmdvel with keyboard control

File: src/ur5_pybullet_ros/script/urdf/ur5_robotiq_85_mobile.urdf (robot description, URDF)
Before this commit: robot ur5_robotiq_85, 25 links, 24 joints
Joints:
- joint chassis_joint: origin xyz=0.0 0.0 0.1 rpy=0.0 0.0 0.0 -> xyz=0.0 0.0 0.06 rpy=0.0 0.0 0.0
- joint lidar_joint: origin xyz=0.2 0.0 0.1 rpy=0.0 0.0 0.0 -> xyz=0.21 0.0 0.06 rpy=0.0 0.0 0.0

File: src/ur5_pybullet_ros/script/urdf/ur5_robotiq_85_mobile_rviz.urdf (robot description, URDF)
Before this commit: robot ur5_robotiq_85, 25 links, 24 joints
Joints:
- joint chassis_joint: origin xyz=0.0 0.0 0.1 rpy=0.0 0.0 0.0 -> xyz=0.0 0.0 0.06 rpy=0.0 0.0 0.0
- joint lidar_joint: origin xyz=0.2 0.0 0.1 rpy=0.0 0.0 0.0 -> xyz=0.21 0.0 0.06 rpy=0.0 0.0 0.0

Commit message: imu ros

File: src/ur5_pybullet_ros/script/urdf/ur5_robotiq_85_mobile.urdf (robot description, URDF)
Before this commit: robot ur5_robotiq_85, 25 links, 24 joints
Links:
- added link imu_link, mass 0
Joints:
- added joint imu_joint: type fixed, parent chassis_link, child imu_link, origin xyz=0.0 0.0 0.0 rpy=0.0 0.0 0.0

File: src/ur5_pybullet_ros/script/urdf/ur5_robotiq_85_mobile_rviz.urdf (robot description, URDF)
Before this commit: robot ur5_robotiq_85, 21 links, 20 joints
Links:
- added link imu_link, mass 0
- link lidar_link: geometry collision cylinder length=0.02 radius=0.03; visual cylinder length=0.02 radius=0.03
Joints:
- added joint imu_joint: type fixed, parent chassis_link, child imu_link, origin xyz=0.0 0.0 0.0 rpy=0.0 0.0 0.0
