Commit message: remove world framefrom  moveit

File: src/ur5_pybullet_ros/script/urdf/ur5_robotiq_85_mobile_rviz.urdf (robot description, URDF)
Before this commit: robot ur5_robotiq_85, 25 links, 24 joints
Links:
- removed link chassis_link_theta
- removed link chassis_link_x
- removed link chassis_link_y
- removed link world
Joints:
- removed joint world_chassis_joint_fixed
- removed joint world_chassis_joint_theta
- removed joint world_chassis_joint_x
- removed joint world_chassis_joint_y

Commit message: moveit planning and navigation with octomap

File: src/ur5_pybullet_ros/script/urdf/ur5_robotiq_85_mobile_rviz.urdf (robot description, URDF)
Before this commit: robot ur5_robotiq_85, 22 links, 21 joints
Links:
- added link world
Joints:
- added joint world_virtual_joint: type floating, parent world, child chassis_link, origin xyz=0 0 0 rpy=0.0 0.0 0, axis 1 0 0, limit lower=-100 upper=100 effort=5000 velocity=3
