Commit message: fake grasp

File: src/ur5_pybullet_ros/script/urdf/objects/ball/green_ball.urdf (robot description, URDF)
Before this commit: robot target, 1 links, 0 joints
Links:
- link base_link: mass 0.1 -> 0.01

File: src/ur5_pybullet_ros/script/urdf/objects/ball/red_ball.urdf (robot description, URDF)
Before this commit: robot target, 1 links, 0 joints
Links:
- link base_link: mass 0.1 -> 0.01

Commit message: better better grasp

File: src/ur5_pybullet_ros/script/urdf/objects/ball/green_ball.urdf (robot description, URDF)
Before this commit: robot ball_green, 1 links, 0 joints
Links:
- link base_link: geometry collision sphere radius=0.03; visual sphere radius=0.03

File: src/ur5_pybullet_ros/script/urdf/objects/ball/red_ball.urdf (robot description, URDF)
Before this commit: robot ball_red, 1 links, 0 joints
Links:
- link base_link: geometry collision sphere radius=0.03; visual sphere radius=0.03
